File: unibody-split/unibody-split.kicad_pcb (KiCad board)
At the start: 2 copper layers, 95 parts, among them IC1 AP130-20, SW1 SW_Push, SW10 SW_Push, SW11 SW_Push, SW12 SW_Push, SW13 SW_Push, SW14 SW_Push, SW15 SW_Push, SW16 SW_Push, SW17 SW_Push, SW18 SW_Push, SW19 SW_Push, SW2 SW_Push, SW20 SW_Push, SW21 SW_Push, SW22 SW_Push, SW23 SW_Push, SW24 SW_Push, SW25 SW_Push, SW26 SW_Push, SW27 SW_Push, SW28 SW_Push, SW29 SW_Push, SW3 SW_Push, SW30 SW_Push, SW31 SW_Push, SW32 SW_Push, SW33 SW_Push, SW34 SW_Push, SW35 SW_Push, SW36 SW_Push, SW37 SW_Push, SW38 SW_Push, SW39 SW_Push, SW4 SW_Push, SW40 SW_Push, SW41 SW_Push, SW42 SW_Push, SW5 SW_Push, SW6 SW_Push, SW7 SW_Push, SW8 SW_Push, SW9 SW_Push, U1 Pico, U2 PMW3360DM-T2QU, U3 HackPackv4-rescue:PSP_1000_JS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

Commit message: Update PCB by adding edge cuts
Parts:
- moved IC1 23.6 mm to (238.8, 149.6), turned to 90 degrees
- moved R1 21.7 mm to (215.3, 149.8), turned to 0 degrees
- moved U1 19.9 mm to (224.8, 108.0)
- moved C2 19.5 mm to (236.2, 159.3)
- moved R2 19.1 mm to (215.3, 155.1), turned to 0 degrees
- moved OL1 17.6 mm to (207.1, 92.9)
- moved SW4 16.9 mm to (254.7, 115.1)
- moved D26 16.9 mm to (315.3, 105.9)
- moved SW41 16.9 mm to (357.5, 130.7)
- moved D10 16.9 mm to (117.4, 125.0)
- moved SW14 16.9 mm to (268.2, 172.0)
- moved D21 16.9 mm to (289.1, 155.4)
- moved D27 16.9 mm to (320.3, 124.3)
- moved D34 16.9 mm to (339.6, 122.8)
- moved SW39 16.9 mm to (347.6, 93.9)
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Other:
- board outline added: 291.5 x 121.9 mm

Commit message: Changed thumb clusters rotation
Parts:
- moved D28 7.34 mm to (161.7, 161.5), turned to 175 degrees
- moved SW28 6.86 mm to (156.9, 169.9), turned to -5 degrees
- moved D21 5.51 mm to (290.4, 160.7), turned to -175 degrees
- moved D35 5.08 mm to (183.5, 166.1), turned to 165 degrees
- moved SW21 4.97 mm to (287.4, 169.7), turned to 5 degrees
- moved D42 4.60 mm to (204.0, 174.5), turned to 155 degrees
- moved U3 4.26 mm to (222.2, 188.1)
- moved SW35 4.09 mm to (177.4, 173.6), turned to -15 degrees
- moved D31 4.08 mm to (170.9, 139.6)
- moved SW29 4.08 mm to (174.7, 110.2)
- moved D32 4.08 mm to (327.1, 89.2)
- moved D10 4.08 mm to (114.8, 128.2)
- moved D11 4.08 mm to (271.0, 100.6)
- moved SW39 4.08 mm to (345.1, 97.0)
- moved OL1 4.08 mm to (204.5, 96.0)
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Other:
- board size 291.5 x 121.9 mm -> 291.5 x 115.4 mm

Commit message: Removed RPi-Pico debug pins, Updated PCB to contain 3 joysticks
Parts:
- added D43: 1N4148, Diode_THT:D_DO-35_SOD27_P7.62mm_Horizontal, B.Cu at (202.6, 183.8)
- added D44: 1N4148, Diode_THT:D_DO-35_SOD27_P7.62mm_Horizontal, B.Cu at (227.2, 191.4)
- added D45: 1N4148, Diode_THT:D_DO-35_SOD27_P7.62mm_Horizontal, B.Cu at (112.7, 161.8)
- added D46: 1N4148, Diode_THT:D_DO-35_SOD27_P7.62mm_Horizontal, B.Cu at (115.8, 150.3)
- added D47: 1N4148, Diode_THT:D_DO-35_SOD27_P7.62mm_Horizontal, B.Cu at (315.1, 157.8)
- added D48: 1N4148, Diode_THT:D_DO-35_SOD27_P7.62mm_Horizontal, B.Cu at (318.2, 169.3)
- added U4: HackPackv4-rescue:PSP_1000_JSTK, HackPack_Footprints:JOYSTICK-PSP1000, F.Cu at (124.8, 162.4)
- added U5: HackPackv4-rescue:PSP_1000_JSTK, HackPack_Footprints:JOYSTICK-PSP1000, F.Cu at (304.0, 162.4)
- moved SW39 7.77 mm to (337.3, 96.5)
- moved U1 7.77 mm to (214.5, 110.6)
- moved SW12 7.77 mm to (266.8, 127.8)
- moved D16 7.77 mm to (131.3, 110.8)
- moved SW10 7.77 mm to (101.0, 135.0)
- moved D19 7.77 mm to (285.7, 110.1)
- moved D18 7.77 mm to (280.8, 91.7)
- moved D35 7.77 mm to (175.7, 165.5)
- moved SW41 7.77 mm to (347.2, 133.3)
- moved D22 7.77 mm to (155.6, 93.9)
- moved SW33 7.77 mm to (322.9, 116.4)
- moved IC1 7.77 mm to (228.4, 146.7)
- moved SW25 7.77 mm to (298.7, 99.6)
- moved SW9 7.77 mm to (105.9, 116.6)
- moved SW32 7.77 mm to (318.0, 98.0)
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Connections:
- U1 pad 17: unconnected-(U1-Pad17) -> joy0
- U1 pad 19: unconnected-(U1-Pad19) -> joy1
- U1 pad 20: unconnected-(U1-Pad20) -> joy2
- U3 pad 1: XIN -> Net-(D43-Pad2)
- U3 pad 2: ADC_VREF -> joy0
- U3 pad 3: YIN -> Net-(D44-Pad2)
Other:
- outline, holes or cut-outs redrawn
